Commit message: Works now with effort control.
Also includes a modified urdf file with reduced mass of the pole part.  The change was needed to debug the Matlab interface.  Now that it works, should probably set back to what it was.

File: urdf/cartpole_gazebo_accel.xacro.urdf (robot description, URDF)
Before this commit: robot cartopole, 4 links, 3 joints
Links:
- link cart: mass 1 -> 5
- link pole: mass 10 -> 1
